Commit message: Added collision hitboxes

File: urdf/arm_4dof.urdf (robot description, URDF)
Before this commit: robot arm_4dof, 5 links, 4 joints
Links:
- added link end_effector; visual mesh filename=4_dof_meshes/end_effector_trans.stl scale=0.01 0.01 0.01
- link arm: geometry collision box size=0.0 0.0 0.0; collision box size=0.125 0.125 0.75
- link base: geometry collision box size=2.0 2.0 0.05; visual mesh filename=4_dof_meshes/base.stl scale=0.01 0.01 0.01
- link forearm: geometry collision box size=0.1 0.15 0.58; visual mesh filename=4_dof_meshes/forearm_trans.stl scale=0.01 0.01 0.01
- link shoulder: geometry collision box size=0.125 0.22 0.25; visual mesh filename=4_dof_meshes/shoulder.stl scale=0.01 0.01 0.01
- link wrist: geometry collision box size=0.125 0.145 0.45; visual mesh filename=4_dof_meshes/wrist_trans.stl scale=0.01 0.01 0.01
Joints:
- added joint wrist_ee: type fixed, parent wrist, child end_effector, origin xyz=0 -0.01 0.6 rpy=0 0 0, axis 1 0 0
- joint joint3_elbow_pitch: limit lower=-2.5 upper=2.5 effort=10 velocity=1 -> lower=-3.14 upper=3.14 effort=10 velocity=1

Commit message: Configured collision geometries

File: urdf/arm_4dof.urdf (robot description, URDF)
Before this commit: robot arm_4dof, 6 links, 5 joints
Links:
- link arm: geometry collision box size=0.125 0.16 1.5; visual mesh filename=4_dof_meshes/arm_trans.stl scale=0.01 0.01 0.01
- link base: geometry collision box size=3.0 3.0 0.08; visual mesh filename=4_dof_meshes/base.stl scale=0.01 0.01 0.01
- link forearm: geometry collision box size=0.1 0.25 1.15; visual mesh filename=4_dof_meshes/forearm_trans.stl scale=0.01 0.01 0.01
- link shoulder: geometry collision box size=0.2 0.35 0.37; visual mesh filename=4_dof_meshes/shoulder.stl scale=0.01 0.01 0.01
- link wrist: geometry collision box size=0.125 0.2 0.8; visual mesh filename=4_dof_meshes/wrist_trans.stl scale=0.01 0.01 0.01
